File: hardware/usb_sniffer_h7p20/usb_sniffer_h7p20.kicad_pcb (KiCad board)
At the start: 4 copper layers, 45 x 45 mm, 141 parts, among them J1 FPGA_JTAG, J2 USB_C_Receptacle_USB2.0_16P, J3 USB_A, J4 USB_C_Receptacle_USB2.0_16P, J5 FFC-40P-0.5mm,NC, J6 Trigger, U1 H7P20N0L128-M3H1, U11 EA3036C, U2 LM2903A-VR, U3 LM2903A-VR, U4 LM2903A-VR, U5 USB3343, U6 P25Q32SH-SSH-IT, U7 CY7C68013A-56LTX, U8 24C64BN, U9 CJ3439KDW, Y2 24M

Commit message: [usb_sniffer_h7p20] production_files.2025620
Routing:
- net GND: track 90.5 -> 89.3 mm, vias 98 -> 97
Other:
- board text added: "USB Sniffer H7P20 20250620"
- board text removed: "USB Sniffer H7P20 20250615"
Changed lines of the file:
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@@
   (gr_arc (start 134 78.5) (mid 134.707107 78.792893) (end 135 79.5)
     (stroke (width 0.05) (type solid)) (layer "Edge.Cuts"))
-  (gr_text "USB Sniffer H7P20\n20250615" (at 119.1006 106.8324) (layer "B.SilkS")
+  (gr_text "USB Sniffer H7P20\n20250620" (at 119.1006 106.8324) (layer "B.SilkS")
     (effects (font (size 1 1) (thickness 0.15)) (justify right bottom mirror))
   )
@@
   (segment (start 95.4818 86.1564) (end 95.4818 85.9314) (width 0.2032) (layer "F.Cu") (net 1))
   (segment (start 108.966 78.105) (end 108.458 78.105) (width 0.127) (layer "F.Cu") (net 1))
-  (segment (start 114.681 92.7354) (end 114.5794 92.6338) (width 0.127) (layer "F.Cu") (net 1))
   (segment (start 103.6978 90.947) (end 103.7082 90.9574) (width 0.3048) (layer "F.Cu") (net 1))
   (segment (start 128.3716 98.0694) (end 128.3716 98.7298) (width 0.5588) (layer "F.Cu") (net 1))
@@
   (segment (start 102.2096 84.3814) (end 102.0546 84.3814) (width 0.2032) (layer "F.Cu") (net 1))
   (segment (start 100.7898 98.6308) (end 100.7872 98.6282) (width 0.3048) (layer "F.Cu") (net 1))
-  (segment (start 114.681 93.726) (end 114.681 92.7354) (width 0.127) (layer "F.Cu") (net 1))
   (segment (start 95.7112 95.881) (end 94.9873 95.881) (width 0.2032) (layer "F.Cu") (net 1))
   (segment (start 111.5728 85.4816) (end 110.2353 85.4816) (width 0.2032) (layer "F.Cu") (net 1))
@@
   (via (at 108.7978 107.4928) (size 0.45212) (drill 0.2032) (layers "F.Cu" "B.Cu") (net 1))
   (via (at 124.333 106.012404) (size 0.45212) (drill 0.2032) (layers "F.Cu" "B.Cu") (free) (net 1))
-  (via (at 114.5794 92.6338) (size 0.45212) (drill 0.2032) (layers "F.Cu" "B.Cu") (net 1))
   (via (at 106.1212 87.2236) (size 0.45212) (drill 0.2032) (layers "F.Cu" "B.Cu") (net 1))
   (via (at 103.7082 90.9574) (size 0.45212) (drill 0.2032) (layers "F.Cu" "B.Cu") (net 1))
@@
   (via (at 109.1593 88.7556) (size 0.45212) (drill 0.2032) (layers "F.Cu" "B.Cu") (net 1))
   (via (at 122.1486 93.614) (size 0.45212) (drill 0.2032) (layers "F.Cu" "B.Cu") (net 1))
-  (via (at 115.2906 91.44) (size 0.45212) (drill 0.2032) (layers "F.Cu" "B.Cu") (free) (net 1))
+  (via (at 115.4176 91.2876) (size 0.45212) (drill 0.2032) (layers "F.Cu" "B.Cu") (free) (net 1))
   (via (at 98.7806 87.9602) (size 0.45212) (drill 0.2032) (layers "F.Cu" "B.Cu") (free) (net 1))
   (via (at 100.5586 95.9612) (size 0.45212) (drill 0.2032) (layers "F.Cu" "B.Cu") (free) (net 1))
@@
   (via (at 116.5606 105.4862) (size 0.45212) (drill 0.2032) (layers "F.Cu" "B.Cu") (net 10))
   (segment (start 116.4 117.2464) (end 114.7744 115.6208) (width 0.5588) (layer "In2.Cu") (net 10))
-  (segment (start 98.933 105.7148) (end 99.1108 105.537) (width 0.9144) (layer "In2.Cu") (net 10))
   (segment (start 103.4034 116.7638) (end 103.4796 116.6876) (width 0.5588) (layer "In2.Cu") (net 10))
   (segment (start 114.7744 115.6208) (end 114.2492 115.6208) (width 0.5588) (layer "In2.Cu") (net 10))
   (segment (start 103.4034 117.6248) (end 103.4034 116.7638) (width 0.5588) (layer "In2.Cu") (net 10))
-  (segment (start 99.1108 105.537) (end 99.1108 101.37648) (width 0.9144) (layer "In2.Cu") (net 10))
-  (segment (start 99.6696 106.4514) (end 98.933 105.7148) (width 0.9144) (layer "In2.Cu") (net 10))
+  (segment (start 119.634 104.4702) (end 117.7798 106.3244) (width 0.5588) (layer "In2.Cu") (net 10))
+  (segment (start 99.6696 111.506) (end 99.6696 106.4514) (width 0.9144) (layer "In2.Cu") (net 10))
   (segment (start 117.7798 112.0902) (end 117.7798 107.188) (width 0.9144) (layer "In2.Cu") (net 10))
   (segment (start 99.6696 111.506) (end 99.6696 112.3696) (width 0.4064) (layer "In2.Cu") (net 10))
-  (segment (start 116.38026 99.36226) (end 119.634 102.616) (width 0.5588) (layer "In2.Cu") (net 10))
   (segment (start 99.6696 111.506) (end 99.3648 111.8108) (width 0.5588) (layer "In2.Cu") (net 10))
   (segment (start 111.7346 116.713) (end 111.7092 116.6876) (width 0.5588) (layer "In2.Cu") (net 10))
@@
   (segment (start 113.1824 116.6876) (end 114.2492 115.6208) (width 0.9144) (layer "In2.Cu") (net 10))
   (segment (start 111.7346 117.6528) (end 111.7346 116.713) (width 0.5588) (layer "In2.Cu") (net 10))
-  (segment (start 119.634 102.616) (end 119.634 104.4702) (width 0.5588) (layer "In2.Cu") (net 10))
   (segment (start 117.348 107.188) (end 117.7798 107.188) (width 0.5588) (layer "In2.Cu") (net 10))
+  (segment (start 113.673483 99.068483) (end 114.1222 99.5172) (width 0.5588) (layer "In2.Cu") (net 10))
   (segment (start 99.06 79.9084) (end 98.5774 79.9084) (width 0.9144) (layer "In2.Cu") (net 10))
-  (segment (start 98.1964 106.0704) (end 98.5774 106.0704) (width 0.5588) (layer "In2.Cu") (net 10))
   (segment (start 106.1212 117.6142) (end 106.1212 116.6876) (width 0.5588) (layer "In2.Cu") (net 10))
   (segment (start 116.5606 105.4862) (end 116.9416 105.4862) (width 0.5588) (layer "In2.Cu") (net 10))
@@
   (segment (start 100.3808 100.0506) (end 99.6188 100.0506) (width 0.4064) (layer "In2.Cu") (net 10))
   (segment (start 106.1278 117.6208) (end 106.1212 117.6142) (width 0.5588) (layer "In2.Cu") (net 10))
-  (segment (start 113.673483 99.068483) (end 113.978283 99.068483) (width 0.5588) (layer "In2.Cu") (net 10))
-  (segment (start 98.5774 106.0704) (end 98.933 105.7148) (width 0.5588) (layer "In2.Cu") (net 10))
-  (segment (start 113.978283 99.068483) (end 114.27206 99.36226) (width 0.5588) (layer "In2.Cu") (net 10))
+  (segment (start 116.5352 99.5172) (end 119.634 102.616) (width 0.5588) (layer "In2.Cu") (net 10))
   (segment (start 99.3648 111.8108) (end 98.4758 111.8108) (width 0.5588) (layer "In2.Cu") (net 10))
   (segment (start 111.7092 116.6876) (end 113.1824 116.6876) (width 0.9144) (layer "In2.Cu") (net 10))
   (segment (start 116.9416 105.4862) (end 117.7798 106.3244) (width 0.5588) (layer "In2.Cu") (net 10))
-  (segment (start 119.634 104.4702) (end 117.7798 106.3244) (width 0.5588) (layer "In2.Cu") (net 10))
+  (segment (start 114.1222 99.5172) (end 116.5352 99.5172) (width 0.5588) (layer "In2.Cu") (net 10))
   (segment (start 106.1212 116.6876) (end 111.7092 116.6876) (width 0.9144) (layer "In2.Cu") (net 10))
+  (segment (start 99.6696 106.4514) (end 99.1108 105.8926) (width 0.9144) (layer "In2.Cu") (net 10))
+  (segment (start 98.933 106.0704) (end 99.1108 105.8926) (width 0.5588) (layer "In2.Cu") (net 10))
+  (segment (start 99.1108 101.37648) (end 99.69754 100.78974) (width 0.9144) (layer "In2.Cu") (net 10))
   (segment (start 99.69754 100.78974) (end 99.69754 80.54594) (width 0.9144) (layer "In2.Cu") (net 10))
-  (segment (start 99.6696 111.506) (end 99.6696 106.4514) (width 0.9144) (layer "In2.Cu") (net 10))
   (segment (start 117.7798 106.3244) (end 117.7798 107.188) (width 0.9144) (layer "In2.Cu") (net 10))
+  (segment (start 98.1964 106.0704) (end 98.933 106.0704) (width 0.5588) (layer "In2.Cu") (net 10))
   (segment (start 99.6696 112.3696) (end 99.4664 112.5728) (width 0.4064) (layer "In2.Cu") (net 10))
-  (segment (start 99.1108 101.37648) (end 99.69754 100.78974) (width 0.9144) (layer "In2.Cu") (net 10))
-  (segment (start 114.27206 99.36226) (end 116.38026 99.36226) (width 0.5588) (layer "In2.Cu") (net 10))
+  (segment (start 119.634 102.616) (end 119.634 104.4702) (width 0.5588) (layer "In2.Cu") (net 10))
+  (segment (start 99.1108 105.8926) (end 99.1108 101.37648) (width 0.9144) (layer "In2.Cu") (net 10))
   (segment (start 114.2492 115.6208) (end 117.7798 112.0902) (width 0.9144) (layer "In2.Cu") (net 10))
   (segment (start 99.6696 112.8776) (end 103.4796 116.6876) (width 0.9144) (layer "In2.Cu") (net 10))
@@
   (via (at 130.3782 90.0938) (size 0.508) (drill 0.3048) (layers "F.Cu" "B.Cu") (net 73))
   (via (at 124.76765 108.7628) (size 0.508) (drill 0.3048) (layers "F.Cu" "B.Cu") (net 73))
-  (segment (start 130.6322 90.0938) (end 131.0005 90.4621) (width 0.9144) (layer "In2.Cu") (net 73))
+  (segment (start 130.9624 102.5652) (end 124.7648 108.7628) (width 0.9144) (layer "In2.Cu") (net 73))
   (segment (start 124.76765 108.7628) (end 124.05645 108.7628) (width 0.9144) (layer "In2.Cu") (net 73))
+  (segment (start 130.9624 90.424) (end 130.9624 102.5652) (width 0.9144) (layer "In2.Cu") (net 73))
+  (segment (start 130.6322 90.0938) (end 130.9624 90.424) (width 0.9144) (layer "In2.Cu") (net 73))
   (segment (start 127.5588 85.5856) (end 127.5588 86.1314) (width 0.9144) (layer "In2.Cu") (net 73))
-  (segment (start 131.0005 102.5271) (end 124.7648 108.7628) (width 0.9144) (layer "In2.Cu") (net 73))
   (segment (start 130.6322 89.2048) (end 130.6322 90.0938) (width 0.9144) (layer "In2.Cu") (net 73))
+  (segment (start 124.7648 108.7628) (end 124.05645 108.7628) (width 0.9144) (layer "In2.Cu") (net 73))
   (segment (start 127.5588 86.1314) (end 130.6322 89.2048) (width 0.9144) (layer "In2.Cu") (net 73))
   (segment (start 127.7112 90.4494) (end 128.4478 90.4494) (width 0.4064) (layer "In2.Cu") (net 73))
   (segment (start 128.4478 90.4494) (end 128.8034 90.0938) (width 0.4064) (layer "In2.Cu") (net 73))
   (segment (start 128.8034 90.0938) (end 130.6322 90.0938) (width 0.4064) (layer "In2.Cu") (net 73))
-  (segment (start 124.7648 108.7628) (end 124.05645 108.7628) (width 0.9144) (layer "In2.Cu") (net 73))
-  (segment (start 131.0005 90.4621) (end 131.0005 102.5271) (width 0.9144) (layer "In2.Cu") (net 73))
   (segment (start 128.5778 89.2356) (end 129.087648 89.2356) (width 0.127) (layer "F.Cu") (net 74))
   (segment (start 129.423248 88.9) (end 130.6068 88.9) (width 0.127) (layer "F.Cu") (net 74))
