File: hardware/usb_sniffer_h7p20/ET3036C.kicad_sch (KiCad schematic)
At the start: 25 parts, among them U11 EA3036C

Commit message: [usb_sniffer_h7p20] CH132C测试无数据，回退USB3343
Parts:
- U11: footprint Package_DFN_QFN:QFN-20-1EP_3x3mm_P0.4mm_EP1.65x1.65mm -> vllogic:QFN-20-1EP_3x3mm_P0.4mm_EP1.65x1.65mm
Changed lines of the file:
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@@
 			)
 		)
-		(property "Footprint" "Package_DFN_QFN:QFN-20-1EP_3x3mm_P0.4mm_EP1.65x1.65mm"
+		(property "Footprint" "vllogic:QFN-20-1EP_3x3mm_P0.4mm_EP1.65x1.65mm"
 			(at 142.24 96.52 0)
 			(effects
