File: hardware/dalishen_pi_h7p20/dalishen_pi_h7p20.kicad_sch (KiCad schematic)
At the start: 99 parts, among them J1 Conn_02x05_Odd_Even, J6 5V, J7 OV5640, J9 D500C930SV0, SW1 SW_Push, SW2 SW_Push, SW3 SW_DIP_x03, SW4 SW_Push, SW5 SW_Push, U3 H7P20N0L128-M3H1, U4 SY7201ABC, U5 XC6206-2.8, U7 P25Q64SH-SSH-IR, U8 XC6206-1.5, X1 NC

Commit message: [dalishen_pi_h7p20] 备份
Connections:
- net B10_IO12N: now also J9.11 (Pin_11); no longer J9.30 (Pin_30)
- net B10_IO12P: now also J9.10 (Pin_10); no longer J9.31 (Pin_31)
- net B10_IO2N: now also J9.23 (Pin_23); no longer J9.18 (Pin_18)
- net B10_IO2P: now also J9.22 (Pin_22); no longer J9.19 (Pin_19)
- net B10_IO4N: now also J9.20 (Pin_20); no longer J9.21 (Pin_21)
- net B10_IO4P: now also J9.19 (Pin_19); no longer J9.22 (Pin_22)
- net B10_IO6N: now also J9.17 (Pin_17); no longer J9.24 (Pin_24)
- net B10_IO6P: now also J9.16 (Pin_16); no longer J9.25 (Pin_25)
- net B10_IO9N: now also J9.14 (Pin_14); no longer J9.27 (Pin_27)
- net B10_IO9P: now also J9.13 (Pin_13); no longer J9.28 (Pin_28)
- net GND: now also J9.15 (Pin_15), J9.18 (Pin_18), J9.21 (Pin_21), J9.24 (Pin_24), J9.33 (Pin_33), J9.38 (Pin_38); no longer J9.17 (Pin_17), J9.20 (Pin_20), J9.23 (Pin_23), J9.26 (Pin_26), J9.3 (Pin_3), J9.8 (Pin_8)
- net LEDA: now also J9.6 (Pin_6), J9.7 (Pin_7); no longer J9.34 (Pin_34), J9.35 (Pin_35)
- net LEDK: now also J9.2 (Pin_2), J9.3 (Pin_3); no longer J9.38 (Pin_38), J9.39 (Pin_39)
- net OV/TP_SCL: now also J9.37 (Pin_37); no longer J9.4 (Pin_4)
- net OV/TP_SDA: now also J9.36 (Pin_36); no longer J9.5 (Pin_5)
- net TP_INT: now also J9.35 (Pin_35); no longer J9.6 (Pin_6)
- net VCC_3V3: now also J9.25 (Pin_25), J9.26 (Pin_26), J9.27 (Pin_27), J9.28 (Pin_28), J9.39 (Pin_39); no longer J9.13 (Pin_13), J9.14 (Pin_14), J9.15 (Pin_15), J9.16 (Pin_16), J9.2 (Pin_2)
- net at R22.1: now also J9.34 (Pin_34); no longer J9.7 (Pin_7)
- net at TP1.1: now also J9.30 (Pin_30); no longer J9.11 (Pin_11)
- net at R21.1: now also J9.31 (Pin_31); no longer J9.10 (Pin_10)
Other:
- moved on the sheet: CY_J1, CY_J2, J6, JP1

Commit message: [dalishen_pi_h7p20] production_files.20250820
Parts:
- J7: footprint Connector_FFC-FPC:Hirose_FH12-24S-0.5SH_1x24-1MP_P0.50mm_Horizontal -> vllogic:Hirose_FH12-24S-0.5SH_1x24-1MP_P0.50mm_Horizontal
- J9: footprint Connector_FFC-FPC:Hirose_FH12-40S-0.5SH_1x40-1MP_P0.50mm_Horizontal -> vllogic:Hirose_FH12-40S-0.5SH_1x40-1MP_P0.50mm_Horizontal
Other:
- note added: "注：JP1短接后可对外输出3.3V。对接EZ-USB板时不要短接。"
- note removed: "注：JP1短接后可对外输出3.3V。EZ-USB板不需要短接。"
Changed lines of the file:
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@@
 		)
 	)
-	(text "注：JP1短接后可对外输出3.3V。EZ-USB板不需要短接。"
+	(text "注：JP1短接后可对外输出3.3V。对接EZ-USB板时不要短接。"
 		(exclude_from_sim no)
 		(at 17.018 275.844 0)
@@
 			(font
 				(face "仿宋")
-				(size 2.54 2.54)
+				(size 2.413 2.413)
 				(thickness 0.6)
 				(bold yes)
@@
 			)
 		)
-		(property "Footprint" "Connector_FFC-FPC:Hirose_FH12-24S-0.5SH_1x24-1MP_P0.50mm_Horizontal"
+		(property "Footprint" "vllogic:Hirose_FH12-24S-0.5SH_1x24-1MP_P0.50mm_Horizontal"
 			(at 288.29 240.03 0)
 			(effects
@@
 			)
 		)
-		(property "Footprint" "Connector_FFC-FPC:Hirose_FH12-40S-0.5SH_1x40-1MP_P0.50mm_Horizontal"
+		(property "Footprint" "vllogic:Hirose_FH12-40S-0.5SH_1x40-1MP_P0.50mm_Horizontal"
 			(at 391.16 227.33 0)
 			(effects

Commit message: [dalishen_pi_h7p20] production_files.20250820 新增保险丝
Parts:
- JP2: footprint Jumper:SolderJumper-2_P1.3mm_Bridged2Bar_RoundedPad1.0x1.5mm -> Jumper:SolderJumper-2_P1.3mm_Bridged_RoundedPad1.0x1.5mm
Changed lines of the file:
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@@
 			)
 		)
-		(property "Footprint" "Jumper:SolderJumper-2_P1.3mm_Bridged2Bar_RoundedPad1.0x1.5mm"
+		(property "Footprint" "Jumper:SolderJumper-2_P1.3mm_Bridged_RoundedPad1.0x1.5mm"
 			(at 335.28 20.32 0)
 			(effects
