File: hardware/dalishen_pi_h7p20/dalishen_pi_h7p20.kicad_sch (KiCad schematic)
At the start: 99 parts, among them J1 Conn_02x05_Odd_Even, J5 OLED_I2C_128x64, J6 NC, J7 OV5640, J9 D500C930SV0, SW1 SW_Push, SW2 SW_Push, SW3 SW_DIP_x03, SW4 SW_Push, SW5 SW_Push, U3 H7P20N0L128-M3H1, U4 SY7201ABC, U5 XC6206-2.8, U7 P25Q64SH-SSH-IR, U8 XC6206-1.5

Commit message: [dalishen_pi_h7p20] 生成方波
Parts:
- removed FID1, FID2, FID3: Fiducial, Fiducial:Fiducial_1mm_Mask2mm, symbol Mechanical:Fiducial
- removed J5: OLED_I2C_128x64, Connector_PinSocket_2.54mm:PinSocket_1x04_P2.54mm_Vertical, symbol Connector_Generic:Conn_01x04
- removed J6: NC, Connector_PinHeader_2.54mm:PinHeader_1x03_P2.54mm_Horizontal, symbol Connector_Generic:Conn_01x03
- removed JP7, JP8: SolderJumper_2_Bridged, Jumper:SolderJumper-2_P1.3mm_Bridged_RoundedPad1.0x1.5mm, symbol Jumper:SolderJumper_2_Bridged
- removed R10: 33, Resistor_SMD:R_0402_1005Metric, symbol Device:R
- removed R14: 470, Resistor_SMD:R_0402_1005Metric, symbol Device:R
- added C2: NC, Capacitor_SMD:C_0402_1005Metric, symbol Device:C
- added CY_J1, CY_J2: Conn_02x10_Odd_Even, Connector_PinSocket_2.54mm:PinSocket_2x10_P2.54mm_Vertical, symbol Connector_Generic:Conn_02x10_Odd_Even
- added J6: 5V, Connector_PinHeader_2.54mm:PinHeader_1x01_P2.54mm_Horizontal, symbol Connector_Generic:Conn_01x01
- added JP1, JP10: SolderJumper_2_Open, Jumper:SolderJumper-2_P1.3mm_Open_RoundedPad1.0x1.5mm, symbol Jumper:SolderJumper_2_Open
- added R16, R23, R25, R26, R27, R28: 2.49k, Resistor_SMD:R_0402_1005Metric, symbol Device:R
- added R7: NC, Resistor_SMD:R_0402_1005Metric, symbol Device:R
- added X1: NC, vllogic:OSC_3225, symbol Oscillator:XO32
- J7: footprint vllogic:Hirose_FH12-24S-0.5SH_1x24-1MP_P0.50mm_Horizontal -> Connector_FFC-FPC:Hirose_FH12-24S-0.5SH_1x24-1MP_P0.50mm_Horizontal
- J9: footprint vllogic:Hirose_FH12-40S-0.5SH_1x40-1MP_P0.50mm_Horizontal -> Connector_FFC-FPC:Hirose_FH12-40S-0.5SH_1x40-1MP_P0.50mm_Horizontal
- JP2: footprint Jumper:SolderJumper-2_P1.3mm_Bridged_RoundedPad1.0x1.5mm -> Jumper:SolderJumper-2_P1.3mm_Bridged2Bar_RoundedPad1.0x1.5mm
- R24: value 33 -> 2.49k
- R8: value 470 -> 33
Connections:
- net KEY3 is gone; now on net KEY2: SW5.1, U3.102 (IO33_MISO3_2)
- net USB334x_SP1/USB334x_26M is gone; now on net FPGA_RX: R24.2
- net USB334x_SP1_D7 is gone; now on an unnamed net: U3.6 (IO13_PCLK_8)
- net B10_IO12N: now also J9.30 (Pin_30); no longer J9.11 (Pin_11)
- net B10_IO12P: now also J9.31 (Pin_31); no longer J9.10 (Pin_10)
- net B10_IO2N: now also J9.18 (Pin_18); no longer J9.23 (Pin_23)
- net B10_IO2P: now also J9.19 (Pin_19); no longer J9.22 (Pin_22)
- net B10_IO4N: now also J9.21 (Pin_21); no longer J9.20 (Pin_20)
- net B10_IO4P: now also J9.22 (Pin_22); no longer J9.19 (Pin_19)
- net B10_IO6N: now also J9.24 (Pin_24); no longer J9.17 (Pin_17)
- net B10_IO6P: now also J9.25 (Pin_25); no longer J9.16 (Pin_16)
- net B10_IO9N: now also J9.27 (Pin_27); no longer J9.14 (Pin_14)
- net B10_IO9P: now also J9.28 (Pin_28); no longer J9.13 (Pin_13)
- net B1_IO_MSEL0_122: now also CY_J2.11 (Pin_11)
- net B1_IO_MSEL1_124: now also CY_J2.9 (Pin_9)
- net B1_IO_MSEL2_125: now also CY_J2.8 (Pin_8)
- net B2_IO_CDONE_105: now also CY_J2.6 (Pin_6), R16.2
- net B9_IO2P: no longer R8.2
- net FPGA_RX: now also JP1.1 (A)
- net FPGA_TCK: now also R27.2
- net FPGA_TDI: now also R28.2
- net FPGA_TDO: now also R25.2
- net FPGA_TMS: now also R26.2
- net FPGA_TX: now also JP10.1 (A), R23.2
- net GND: now also J9.17 (Pin_17), J9.20 (Pin_20), J9.23 (Pin_23), J9.26 (Pin_26), J9.3 (Pin_3), J9.8 (Pin_8), C2.1, CY_J1.11 (Pin_11), CY_J1.19 (Pin_19), CY_J1.4 (Pin_4), CY_J1.6 (Pin_6), CY_J1.9 (Pin_9), X1.2 (GND); no longer J9.15 (Pin_15), J9.18 (Pin_18), J9.21 (Pin_21), J9.24 (Pin_24), J9.33 (Pin_33), J9.38 (Pin_38)
- net KEY1: now also SW4.1, U3.104 (IO27_GCLK_2); no longer SW1.1, U3.126 (IO3_8)
- net KEY2: no longer SW4.1, U3.104 (IO27_GCLK_2)
- net LEDA: now also J9.34 (Pin_34), J9.35 (Pin_35); no longer J9.6 (Pin_6), J9.7 (Pin_7)
- net LEDK: now also J9.38 (Pin_38), J9.39 (Pin_39); no longer J9.2 (Pin_2), J9.3 (Pin_3)
- net OV/TP_SCL: now also J9.4 (Pin_4); no longer J9.37 (Pin_37)
- net OV/TP_SDA: now also J9.5 (Pin_5); no longer J9.36 (Pin_36)
- net TP_INT: now also J9.6 (Pin_6); no longer J9.35 (Pin_35)
- net VCC_3V3: now also J9.13 (Pin_13), J9.14 (Pin_14), J9.15 (Pin_15), J9.16 (Pin_16), J9.2 (Pin_2), SW3.1, SW3.2, SW3.3, C2.2, R7.1, X1.4 (V+); no longer J9.25 (Pin_25), J9.26 (Pin_26), J9.27 (Pin_27), J9.28 (Pin_28), J9.39 (Pin_39), SW3.4, SW3.5, SW3.6
- net VCC_5V: now also J6.1 (Pin_1)
- net vllinkmodule/VL_RX: now also JP10.2 (B)
- net vllinkmodule/VL_TX: now also JP1.2 (B)
- net at R22.1: now also J9.7 (Pin_7); no longer J9.34 (Pin_34)
- net at TP1.1: now also J9.11 (Pin_11); no longer J9.30 (Pin_30)
- net at R21.1: now also J9.10 (Pin_10); no longer J9.31 (Pin_31)
- net at R57.1: now also SW3.6; no longer SW3.3
- net at R56.1: now also SW3.5; no longer SW3.2
- net at R55.1: now also SW3.4; no longer SW3.1
- net USB334x_SP1_C/R renamed CY_IFCLK
- net CY_IFCLK: now also CY_J1.12 (Pin_12)
- net USB334x_SP1_D0 renamed CY_FD_15
- net CY_FD_15: now also CY_J1.3 (Pin_3)
- net USB334x_SP1_D1 renamed CY_FD_14
- net CY_FD_14: now also CY_J1.2 (Pin_2)
- net USB334x_SP1_D2 renamed CY_FD_13
- net CY_FD_13: now also CY_J1.1 (Pin_1)
- net USB334x_SP1_D3 renamed CY_FD_0
- net CY_FD_0: now also CY_J1.15 (Pin_15)
- net USB334x_SP1_D4 renamed CY_FD_1
- net CY_FD_1: now also CY_J1.16 (Pin_16)
- net USB334x_SP1_D5 renamed CY_FD_2
- net CY_FD_2: now also CY_J1.17 (Pin_17)
- net USB334x_SP1_D6 renamed CY_FD_3
- net CY_FD_3: now also CY_J1.18 (Pin_18)
- net USB334x_SP1_DIR renamed CY_FD_12
- net CY_FD_12: now also CY_J2.1 (Pin_1)
- net USB334x_SP1_NXT renamed CY_SLWR
- net CY_SLWR: now also CY_J1.8 (Pin_8)
- net USB334x_SP1_STP renamed CY_FD_11
- net CY_FD_11: now also CY_J2.2 (Pin_2)
- net USB334x_SP2_C/R renamed CY_PA1
- net CY_PA1: now also CY_J2.12 (Pin_12)
- net USB334x_SP2_D0 renamed CY_PKTEND
- net CY_PKTEND: now also CY_J2.7 (Pin_7)
- net USB334x_SP2_D1 renamed CY_FD_8
- net CY_FD_8: now also CY_J2.5 (Pin_5)
- net USB334x_SP2_D2 renamed CY_FD_9
- net CY_FD_9: now also CY_J2.4 (Pin_4)
- net USB334x_SP2_D3 renamed CY_FD_6
- net CY_FD_6: now also CY_J2.18 (Pin_18)
- net USB334x_SP2_D4 renamed CY_FD_7
- net CY_FD_7: now also CY_J2.17 (Pin_17)
- net USB334x_SP2_D5 renamed CY_FLAGB
- net CY_FLAGB: now also CY_J2.15 (Pin_15)
- net USB334x_SP2_D6 renamed CY_SLRD
- net CY_SLRD: now also CY_J1.7 (Pin_7)
- net USB334x_SP2_D7 renamed CY_PA0
- net CY_PA0: now also CY_J2.13 (Pin_13)
- net USB334x_SP2_DIR renamed CY_FD_5
- net CY_FD_5: now also CY_J2.19 (Pin_19)
- net USB334x_SP2_NXT renamed CY_PA3
- net CY_PA3: now also CY_J2.10 (Pin_10)
- net USB334x_SP2_STP renamed CY_FD_4
- net CY_FD_4: now also CY_J2.20 (Pin_20)
- net USB334x_SPx_26M renamed CY_FD_10
- net CY_FD_10: now also CY_J2.3 (Pin_3); no longer R24.1
- new net: R7.2, X1.1 (EN)
- new net: R8.2, X1.3 (OUT)
- new net CY_FLAGA: CY_J2.16 (Pin_16), R16.1
- new net CY_FLAGC: CY_J2.14 (Pin_14)
- new net KEY0: SW1.1, U3.126 (IO3_8)
- new net USB20_DM_CMP1: R28.1
- new net USB20_DM_CMP2: R26.1
- new net USB20_DM_CMP3: R24.1
- new net USB20_DP_CMP1: R27.1
- new net USB20_DP_CMP2: R25.1
- new net USB20_DP_CMP3: R23.1
- no-connect marks 12 -> 18
Other:
- removed sheet USB334x_SP1
- removed sheet USB334x_SP2
- sheet USB334x ports: added USB20_DM_CMP1, USB20_DM_CMP2, USB20_DM_CMP3, USB20_DP_CMP1, USB20_DP_CMP2, USB20_DP_CMP3; removed none
- note added: "EZ-USB CY7C68013A板 对接口（顶对顶） 若68013板已焊排针，本板需焊双排母对接"
- note added: "PD3 PD1 PA7 PA5 PA3 PA1 CTL2 CTL0 PB6 PB4"
- note added: "PD4 PD2 PD0 PA6 PA4 PA2 PA0 CTL1 PB7 PB5"
- note added: "PD5 PD7 CLK RDY0 GND GND SCL PB0 PB2 GND"
- note added: "PD6 GND GND RDY1 VCC IFCLK SDA PB1 PB3 VCC"
- note removed: "0.96寸 I2C OLED 屏幕模块接口"
- moved on the sheet: C10, C11, C16, C17, C18, C19, C20, C21, C22, C23, C24, C38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
