File: hardware/dalishen_pi_h7p20/USB334x_SP.kicad_sch (KiCad schematic)
At the start: 12 parts, among them J2 USB_C_Receptacle_USB2.0_16P, U20 USB3343

Commit message: [dalishen_pi_h7p20] Backup
Parts:
- removed R4: 0, Resistor_SMD:R_0402_1005Metric, symbol Device:R
- renumbered C13 to C1, C15 to C2, C49 to C3, C50 to C80, J2 to J4, R76 to R1, R89 to R12, R90 to R13, R77 to R2, R79 to R3, U20 to U2
Connections:
- net at C80.2, U2.15 (VDD33): now also U2.18 (ID)

Commit message: [dalishen_pi_h7p20] Backup
Parts:
- added F2: SMD0805B100TFT, Fuse:Fuse_0805_2012Metric, symbol Device:Polyfuse
Connections:
- net VCC_5V: now also F2.1; no longer J4.A4 (VBUS), J4.A9 (VBUS), J4.B4 (VBUS), J4.B9 (VBUS)
- new net: F2.2, J4.A4 (VBUS), J4.A9 (VBUS), J4.B4 (VBUS), J4.B9 (VBUS)
Changed lines of the file:
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@@
+	(wire
+		(pts
+			(xy 137.16 53.34) (xy 146.05 53.34)
+		)
+		(stroke
+			(width 0)
+			(type default)
+		)
+	)
 	(wire
 		(pts
@@
 	(wire
 		(pts
-			(xy 116.84 53.34) (xy 146.05 53.34)
+			(xy 116.84 53.34) (xy 129.54 53.34)
 		)
 		(stroke
@@
 					(unit 1)
 				)
+			)
+		)
+	)
+	(symbol
+		(lib_id "Device:Polyfuse")
+		(at 133.35 53.34 270)
+		(unit 1)
+		(exclude_from_sim no)
+		(in_bom yes)
+		(on_board yes)
+		(dnp no)
+		(property "Reference" "F2"
+			(at 133.35 47.625 90)
+			(effects
+				(font
+					(size 1.27 1.27)
+				)
+			)
+		)
+		(property "Value" "SMD0805B100TFT"
+			(at 133.35 49.9364 90)
+			(effects
+				(font
+					(size 1.27 1.27)
+				)
+			)
+		)
+		(property "Footprint" "Fuse:Fuse_0805_2012Metric"
+			(at 128.27 54.61 0)
+			(effects
+				(font
+					(size 1.27 1.27)
+				)
+				(justify left)
+				(hide yes)
+			)
+		)
+		(property "Datasheet" "~"
+			(at 133.35 53.34 0)
+			(effects
+				(font
+					(size 1.27 1.27)
+				)
+				(hide yes)
+			)
+		)
+		(property "Description" ""
+			(at 133.35 53.34 0)
+			(effects
+				(font
+					(size 1.27 1.27)
+				)
+			)
+		)
+		(pin "1"
+		)
+		(pin "2"
+		)
+		(instances
+			(project "dalishen_pi_h7p20"
+				(path "/221176f3-b6da-4f04-afa6-f8c6dd49907a/904b7fed-0faa-4294-9b84-cad3aa7e6c05"
+					(reference "F2")
+					(unit 1)
+				)
+				(path "/221176f3-b6da-4f04-afa6-f8c6dd49907a/c2aa1832-0dff-4f01-98a8-0a8751ca7a00"
+					(reference "F3")
+					(unit 1)
+				)

Commit message: [dalishen_pi_h7p20] 待review
Parts:
- added R27, R66: 0, Resistor_SMD:R_0402_1005Metric, symbol Device:R
- added R37: NC, Resistor_SMD:R_0402_1005Metric, symbol Device:R
- added R59: 10k,1%, Resistor_SMD:R_0402_1005Metric, symbol Device:R
- R13: value 10k,1% -> NC
- U2: footprint Package_DFN_QFN:QFN-24-1EP_4x4mm_P0.5mm_EP2.6x2.6mm -> vllogic:QFN-24-1EP_4x4mm_P0.5mm_EP2.6x2.6mm
Connections:
- net GND: now also R59.2
- net VCC_3V3: now also R27.2
- net at R13.2, U2.22 (~{RESETB}): now also R59.1, R66.2
- net USB334x_CLK: no longer names the net of U2.2 (CLKOUT)
- net USB334x_CLK: now also R27.1, R37.1
- new net USB334x_C/R: R37.2, R66.1
