File: hardware/dalishen_pi_h7p20/ET3036C_CJ3439KDW.kicad_sch (KiCad schematic)
At the start: 29 parts, among them U6 EA3036C, U9 CJ3439KDW

Commit message: [dalishen_pi_h7p20] production_files.20250820
Parts:
- L3, L4, L5: footprint vllogic:L_NR3015 -> vllogic:L_NR2520xx
- U6: footprint Package_DFN_QFN:QFN-20-1EP_3x3mm_P0.4mm_EP1.65x1.65mm -> vllogic:QFN-20-1EP_3x3mm_P0.4mm_EP1.65x1.65mm
Changed lines of the file:
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@@
 			)
 		)
-		(property "Footprint" "vllogic:L_NR3015"
+		(property "Footprint" "vllogic:L_NR2520xx"
 			(at 54.61 17.78 0)
 			(effects
@@
 			)
 		)
-		(property "Footprint" "vllogic:L_NR3015"
+		(property "Footprint" "vllogic:L_NR2520xx"
 			(at 58.42 78.74 0)
 			(effects
@@
 			)
 		)
-		(property "Footprint" "vllogic:L_NR3015"
+		(property "Footprint" "vllogic:L_NR2520xx"
 			(at 90.17 58.42 0)
 			(effects
@@
 			)
 		)
-		(property "Footprint" "Package_DFN_QFN:QFN-20-1EP_3x3mm_P0.4mm_EP1.65x1.65mm"
+		(property "Footprint" "vllogic:QFN-20-1EP_3x3mm_P0.4mm_EP1.65x1.65mm"
 			(at 63.5 53.34 0)
 			(effects

Commit message: [dalishen_pi_h7p20] 生成方波
Parts:
- L3, L4, L5: footprint vllogic:L_NR2520xx -> vllogic:L_NR3015
- U6: footprint vllogic:QFN-20-1EP_3x3mm_P0.4mm_EP1.65x1.65mm -> Package_DFN_QFN:QFN-20-1EP_3x3mm_P0.4mm_EP1.65x1.65mm
